File: FT/kicad/Display Example/Display_example.kicad_pcb (KiCad board)
At the start: 2 copper layers, 53.3 x 54.6 mm, 25 parts, among them J1 Conn_01x07_Male, Q1 Q_PNP_BCE, Q2 Q_PNP_BCE, Q3 Q_PNP_BCE, Q4 Q_PNP_BCE, U1 HDSP-7501, U2 HDSP-7501, U3 HDSP-7501, U4 HDSP-7501

Commit message: KiCad update
Parts:
- removed J1: Conn_01x07_Male, Connector_PinHeader_2.54mm:PinHeader_1x07_P2.54mm_Vertical
- added J2: Conn_01x07_Socket, Connector_PinSocket_2.54mm:PinSocket_1x07_P2.54mm_Vertical, F.Cu at (22.9, 20.3)
