File: FT/kicad/Display Example/Display_example.kicad_sch (KiCad schematic)
At the start: 1 part, among them J1 Conn_01x07_Male

Commit message: KiCad update
Parts:
- removed J1: Conn_01x07_Male, Connector_PinHeader_2.54mm:PinHeader_1x07_P2.54mm_Vertical, symbol Connector:Conn_01x07_Male
- added J2: Conn_01x07_Socket, Connector_PinSocket_2.54mm:PinSocket_1x07_P2.54mm_Vertical, symbol Connector:Conn_01x07_Socket
Connections:
- net CLOCK: now also J2.1 (Pin_1)
- net DATA1: now also J2.2 (Pin_2)
- net DATA2: now also J2.3 (Pin_3)
- net DATA3: now also J2.4 (Pin_4)
- net DATA4: now also J2.5 (Pin_5)
- net GND: now also J2.7 (Pin_7)
- net VCC: now also J2.6 (Pin_6)
