File: FT/kicad/Display Example/display.kicad_sch (KiCad schematic)
At the start: 24 parts, among them Q1 Q_PNP_BCE, Q2 Q_PNP_BCE, Q3 Q_PNP_BCE, Q4 Q_PNP_BCE, U1 HDSP-7501, U2 HDSP-7501, U3 HDSP-7501, U4 HDSP-7501

Commit message: KiCad update
Other:
- moved on the sheet: R12, R2
